Commit message: rename lidar_link to base_scan

File: urdf/two_wheel_mr.urdf (robot description, URDF)
Before this commit: robot two_wheel_mr, 13 links, 12 joints
Links:
- removed link lidar_link
- added link base_scan; collision mesh filename=package://two_wheel_mr/meshes/rplidar.dae scale=0.001 0.001 0.001; visual mesh filename=package://two_wheel_mr/meshes/rplidar.dae scale=0.001 0.001 0.001
Joints:
- joint lidar_joint: child lidar_link -> base_scan
