Commit message: update robot model
no arm yet

File: urdf/robot_description.urdf.xacro (robot description, xacro)
@@ -2,344 +2,632 @@
 <robot xmlns:xacro="http://www.ros.org/wiki/xacro">
   <xacro:macro name="robot" params="prefix">
-    <link name="${prefix}base_link">
-      <inertial>
-      <origin xyz="0.00116919992599684 2.964698431418E-06 0.158519577597417" rpy="0 0 0" />
-      <mass value="78.0827274144149" />
-      <inertia ixx="2.50667109850897" ixy="0.0167986143339606" ixz="-0.00462248899685703"
-           iyy="4.2145346225938" iyz="0.000106887843698203" izz="6.28232013006863" />
-      </inertial>
-      <visual>
-      <origin xyz="0 0 0" rpy="0 0 0" />
-      <geometry>
-        <mesh filename="package://two_wheel_mr/meshes/base.STL" />
-      </geometry>
-      <material name="">
-        <color rgba="0.650980392156863 0.619607843137255 0.588235294117647 1" />
-      </material>
-      </visual>
-      <collision>
-      <origin xyz="0 0 0" rpy="0 0 0" />
-      <geometry>
-        <mesh filename="package://two_wheel_mr/meshes/base.STL" />
-      </geometry>
+    <link
+      name="${prefix}base_link">
+      <inertial>
+        <origin
+          xyz="-0.0152000946909854 0.00117474039315474 0.0910195561515633"
+          rpy="0 0 0" />
+        <mass
+          value="64.5439245165624" />
+        <inertia
+          ixx="1.49121577423484"
+          ixy="-0.000190337575366599"
+          ixz="0.0394039846606287"
+          iyy="3.87052073855067"
+          iyz="0.000421606962278842"
+          izz="5.03992806522733" />
+      </inertial>
+      <visual>
+        <origin
+          xyz="0 0 0"
+          rpy="0 0 0" />
+        <geometry>
+          <mesh
+            filename="package://two_wheel_mr/meshes/base_link.STL" />
+        </geometry>
+        <material
+          name="">
+          <color
+            rgba="1 1 1 1" />
+        </material>
+      </visual>
+      <collision>
+        <origin
+          xyz="0 0 0"
+          rpy="0 0 0" />
+        <geometry>
+          <mesh
+            filename="package://two_wheel_mr/meshes/base_link.STL" />
+        </geometry>
       </collision>
     </link>
     <link name="${prefix}base_footprint" />
     <joint name="${prefix}base_joint" type="fixed">
-      <parent link="${prefix}base_footprint" />
-      <child link="${prefix}base_link" />
+      <parent link="${prefix}${prefix}base_footprint" />
+      <child link="${prefix}${prefix}base_link" />
       <origin xyz="0 0 0" rpy="0 0 0" />
     </joint>
-    <link name="${prefix}left_wheel_link">
-      <inertial>
-      <origin xyz="6.3527E-07 6.4052E-06 8.8161E-06" rpy="0 0 0" />
-      <mass value="0.3265" />
-      <inertia ixx="0.00067921" ixy="2.1629E-18" ixz="1.2457E-17"
-           iyy="0.00038694" iyz="3.8673E-10" izz="0.00038694" />
-      </inertial>
-      <visual>
-      <origin xyz="0 0 0" rpy="0 0 0" />
-      <geometry>
-        <mesh filename="package://two_wheel_mr/meshes/lchinh1.STL" />
-      </geometry>
-      <material name="">
-        <color rgba="0.50196 0.50196 0.50196 1" />
-      </material>
-      </visual>
-      <collision>
-      <origin xyz="0 0 0" rpy="0 0 0" />
-      <geometry>
-        <mesh filename="package://two_wheel_mr/meshes/lchinh1.STL" />
-      </geometry>
-      </collision>
-    </link>
-    <joint name="${prefix}left_wheel_joint" type="continuous">
-      <origin xyz="0 0.21908 0.062877" rpy="1.5708 0.0030806 1.5708" />
-      <parent link="${prefix}base_link" />
-      <child link="${prefix}left_wheel_link" />
-      <axis xyz="1 0 0" />
-    </joint>
-    <link name="${prefix}right_wheel_link">
-      <inertial>
-      <origin xyz="6.3527E-07 4.0168E-06 1.013E-05" rpy="0 0 0" />
-      <mass value="0.3265" />
-      <inertia ixx="0.00067921" ixy="7.1118E-18" ixz="9.5532E-18"
-           iyy="0.00038694" iyz="2.7867E-10" izz="0.00038694" />
-      </inertial>
-      <visual>
-      <origin xyz="0 0 0" rpy="0 0 0" />
-      <geometry>
-        <mesh filename="package://two_wheel_mr/meshes/lchinh2.STL" />
-      </geometry>
-      <material name="">
-        <color rgba="0.50196 0.50196 0.50196 1" />
-      </material>
-      </visual>
-      <collision>
-      <origin xyz="0 0 0" rpy="0 0 0" />
-      <geometry>
-        <mesh filename="package://two_wheel_mr/meshes/lchinh2.STL" />
-      </geometry>
-      </collision>
-    </link>
-    <joint name="${prefix}right_wheel_joint" type="continuous">
-      <origin xyz="0 -0.21908 0.062877" rpy="2.0284 -0.0030806 1.5708" />
-      <parent link="${prefix}base_link" />
-      <child link="${prefix}right_wheel_link" />
-      <axis xyz="0.99998 -0.0055274 0.0027218" />
-    </joint>
-    <link name="${prefix}caster1_wheel_link">
-      <inertial>
-      <origin xyz="0.00946264375129513 -0.0176723960529895 -0.00608687345053327" rpy="0 0 0" />
-      <mass value="0.0812397412253748" />
-      <inertia ixx="7.05605896099002E-05" ixy="4.67952096548945E-07" ixz="-6.32104020706617E-06"
-           iyy="0.000101227602264477" iyz="-3.01006512726596E-07" izz="6.47999500417815E-05" />
-      </inertial>
-      <visual>
-      <origin xyz="0 0 0" rpy="0 0 0" />
-      <geometry>
-        <mesh filename="package://two_wheel_mr/meshes/lbphu1.STL" />
-      </geometry>
-      <material name="">
-        <color rgba="0.686274509803922 0.658823529411765 0.63921568627451 1" />
-      </material>
-      </visual>
-      <collision>
-      <origin xyz="0 0 0" rpy="0 0 0" />
-      <geometry>
-        <mesh filename="package://two_wheel_mr/meshes/lbphu1.STL" />
-      </geometry>
-      </collision>
-    </link>
-    <joint name="${prefix}caster1_wheel_joint" type="fixed">
-      <origin xyz="0.31938 0.18313 0.0747" rpy="1.5708 0 1.5708" />
-      <parent link="${prefix}base_link" />
-      <child link="${prefix}caster1_wheel_link" />
-      <axis xyz="0 -1 0" />
-    </joint>
-    <link name="${prefix}caster1_link">
-      <inertial>
-      <origin xyz="0.0119989443232924 1.70501568419468E-09 -1.61823893174429E-09" rpy="0 0 0" />
-      <mass value="0.0588561914547071" />
-      <inertia ixx="2.10634561244654E-05" ixy="2.9837515375904E-14" ixz="1.48354974680888E-14"
-           iyy="1.38903083736938E-05" iyz="-1.50091507401853E-12" izz="1.38903088244573E-05" />
-      </inertial>
-      <visual>
-      <origin xyz="0 0 0" rpy="0 0 0" />
-      <geometry>
-        <mesh filename="package://two_wheel_mr/meshes/lphu1.STL" />
-      </geometry>
-      <material name="">
-        <color rgba="1 1 1 1" />
-      </material>
-      </visual>
-      <collision>
-      <origin xyz="0 0 0" rpy="0 0 0" />
-      <geometry>
-        <mesh filename="package://two_wheel_mr/meshes/lphu1.STL" />
-      </geometry>
-      </collision>
-    </link>
-    <joint name="${prefix}caster1_joint" type="fixed">
-      <origin xyz="-0.024995 -0.049695 0.0018095" rpy="0 -0.99918 0" />
-      <parent link="${prefix}caster1_wheel_link" />
-      <child link="${prefix}caster1_link" />
-      <axis xyz="-1 0 0" />
-    </joint>
-    <link name="${prefix}caster2_wheel_link">
-      <inertial>
-      <origin xyz="-0.0112512989675595 0.03267239615527 4.39991287848329E-09" rpy="0 0 0" />
-      <mass value="0.0812397511313111" />
-      <inertia ixx="7.46266281902283E-05" ixy="5.56405620269323E-07" ixz="1.05535643802289E-11"
-           iyy="0.00010122761651701" iyz="-6.77914973369374E-12" izz="6.0733928293755E-05" />
-      </inertial>
-      <visual>
-      <origin xyz="0 0 0" rpy="0 0 0" />
-      <geometry>
-        <mesh filename="package://two_wheel_mr/meshes/lbphu2.STL" />
-      </geometry>
-      <material name="">
-        <color rgba="0.686274509803922 0.658823529411765 0.63921568627451 1" />
-      </material>
-      </visual>
-      <collision>
-      <origin xyz="0 0 0" rpy="0 0 0" />
-      <geometry>
-        <mesh filename="package://two_wheel_mr/meshes/lbphu2.STL" />
-      </geometry>
-      </collision>
-    </link>
-    <joint name="${prefix}caster2_wheel_joint" type="fixed">
-      <origin xyz="0.31938 -0.18288 0.0897" rpy="-1.5708 0 -0.57871" />
-      <parent link="${prefix}base_link" />
-      <child link="${prefix}caster2_wheel_link" />
-      <axis xyz="0 1 0" />
-    </joint>
-    <link name="${prefix}caster2_link">
-      <inertial>
-      <origin xyz="-0.0120010556766208 1.70501079921337E-09 -1.62239932599562E-09" rpy="0 0 0" />
-      <mass value="0.0588561914546423" />
-      <inertia ixx="2.1063456124443E-05" ixy="2.98257335018538E-14" ixz="1.55663695875061E-14"
-           iyy="1.38903083736981E-05" iyz="-1.50091476570755E-12" izz="1.38903088244611E-05" />
-      </inertial>
-      <visual>
-      <origin xyz="0 0 0" rpy="0 0 0" />
-      <geometry>
-        <mesh filename="package://two_wheel_mr/meshes/lphu2.STL" />
-      </geometry>
-      <material name="">
-        <color rgba="1 1 1 1" />
-      </material>
-      </visual>
-      <collision>
-      <origin xyz="0 0 0" rpy="0 0 0" />
-      <geometry>
-        <mesh filename="package://two_wheel_mr/meshes/lphu2.STL" />
-      </geometry>
-      </collision>
-    </link>
-    <joint name="${prefix}caster2_joint" type="fixed">
-      <origin xyz="0.022 0.064695 0.012" rpy="0 -1.5708 0" />
-      <parent link="${prefix}caster2_wheel_link" />
-      <child link="${prefix}caster2_link" />
-      <axis xyz="-1 0 0" />
-    </joint>
-    <link name="${prefix}caster3_wheel_link">
-      <inertial>
-      <origin xyz="-0.0112512987405764 0.0326723959483828 3.88080700908233E-09" rpy="0 0 0" />
-      <mass value="0.0812397536824839" />
-      <inertia ixx="7.46266289376794E-05" ixy="5.56405684377692E-07" ixz="1.21728790969442E-11"
-           iyy="0.000101227619883743" iyz="-6.77973950305887E-12" izz="6.07339310000421E-05" />
-      </inertial>
-      <visual>
-      <origin xyz="0 0 0" rpy="0 0 0" />
-      <geometry>
-        <mesh filename="package://two_wheel_mr/meshes/lbphu3.STL" />
-      </geometry>
-      <material name="">
-        <color rgba="0.686274509803922 0.658823529411765 0.63921568627451 1" />
-      </material>
-      </visual>
-      <collision>
-      <origin xyz="0 0 0" rpy="0 0 0" />
-      <geometry>
-        <mesh filename="package://two_wheel_mr/meshes/lbphu3.STL" />
-      </geometry>
-      </collision>
-    </link>
-    <joint name="${prefix}caster3_wheel_joint" type="fixed">
-      <origin xyz="-0.31863 0.18313 0.0897" rpy="-1.5708 0 3.1416" />
-      <parent link="${prefix}base_link" />
-      <child link="${prefix}caster3_wheel_link" />
-      <axis xyz="0 1 0" />
-    </joint>
-    <link name="${prefix}caster3_link">
-      <inertial>
-      <origin xyz="0.0119999999999998 -2.21784146603454E-10 -3.31598748459783E-10" rpy="0 0 0" />
-      <mass value="0.0588561914567127" />
-      <inertia ixx="2.10634561252174E-05" ixy="1.35878504384566E-14" ixz="-9.08799413589546E-15"
-           iyy="1.38903090958169E-05" iyz="-1.20252769127507E-12" izz="1.38903081021528E-05" />
-      </inertial>
-      <visual>
-      <origin xyz="0 0 0" rpy="0 0 0" />
-      <geometry>
-        <mesh filename="package://two_wheel_mr/meshes/lphu3.STL" />
-      </geometry>
-      <material name="">
-        <color rgba="0.250980392156863 0.250980392156863 0.250980392156863 1" />
-      </material>
-      </visual>
-      <collision>
-      <origin xyz="0 0 0" rpy="0 0 0" />
-      <geometry>
-        <mesh filename="package://two_wheel_mr/meshes/lphu3.STL" />
-      </geometry>
-      </collision>
-    </link>
-    <joint name="${prefix}caster3_joint" type="fixed">
-      <origin xyz="0.022 0.064695 -0.012" rpy="1.9626 -1.5708 0" />
-      <parent link="${prefix}caster3_wheel_link" />
-      <child link="${prefix}caster3_link" />
-      <axis xyz="-1 0 0" />
-    </joint>
-    <link name="${prefix}caster4_wheel_link">
-      <inertial>
-      <origin xyz="-0.00013615031454986 -0.017672396198252 -0.0112504775096143" rpy="0 0 0" />
-      <mass value="0.0812397612278049" />
-      <inertia ixx="6.07359732393891E-05" ixy="-6.72855516700748E-09" ixz="1.6810978297091E-07"
-           iyy="0.000101227631072605" iyz="-5.56367639975508E-07" izz="7.46246003421395E-05" />
-      </inertial>
-      <visual>
-      <origin xyz="0 0 0" rpy="0 0 0" />
-      <geometry>
-        <mesh filename="package://two_wheel_mr/meshes/lbphu4.STL" />
-      </geometry>
-      <material name="">
-        <color rgba="0.792156862745098 0.819607843137255 0.933333333333333 1" />
-      </material>
-      </visual>
-      <collision>
-      <origin xyz="0 0 0" rpy="0 0 0" />
-      <geometry>
-        <mesh filename="package://two_wheel_mr/meshes/lbphu4.STL" />
-      </geometry>
-      </collision>
-    </link>
-    <joint name="${prefix}caster4_wheel_joint" type="fixed">
-      <origin xyz="-0.31863 -0.18288 0.0747" rpy="1.5708 0 1.5708" />
-      <parent link="${prefix}base_link" />
-      <child link="${prefix}caster4_wheel_link" />
-      <axis xyz="0 -1 0" />
-    </joint>
-    <link name="${prefix}caster4_link">
-      <inertial>
-      <origin xyz="-0.0120010556442718 3.15797032968135E-09 -1.62441360362919E-09" rpy="0 0 0" />
-      <mass value="0.0588561914225415" />
-      <inertia ixx="2.1063456114227E-05" ixy="-2.253105819105E-13" ixz="1.10871181094577E-14"
-           iyy="1.38903083735561E-05" iyz="-1.50168295974446E-12" izz="1.38903088255762E-05" />
-      </inertial>
-      <visual>
-      <origin xyz="0 0 0" rpy="0 0 0" />
-      <geometry>
-        <mesh filename="package://two_wheel_mr/meshes/lphu4.STL" />
-      </geometry>
-      <material name="">
-        <color rgba="0.250980392156863 0.250980392156863 0.250980392156863 1" />
-      </material>
-      </visual>
-      <collision>
-      <origin xyz="0 0 0" rpy="0 0 0" />
-      <geometry>
-        <mesh filename="package://two_wheel_mr/meshes/lphu4.STL" />
-      </geometry>
-      </collision>
-    </link>
-    <joint name="${prefix}caster4_joint" type="fixed">
-      <origin xyz="0.012265 -0.049695 0.021853" rpy="1.5708 0.012101 0" />
-      <parent link="${prefix}caster4_wheel_link" />
-      <child link="${prefix}caster4_link" />
-      <axis xyz="-1 0 0" />
-    </joint>
-    <link name="${prefix}lidar_link">
-      <visual>
-      <origin xyz="0.0 0.0 0.0" rpy="1.5707 0 4.71" />
-      <geometry>
-        <mesh filename="package://two_wheel_mr/meshes/rplidar.dae" scale="0.001 0.001 0.001" />
-      </geometry>
-      <material name="LightGrey">
-        <color rgba="0.7 0.7 0.7 1.0" />
-      </material>
-      </visual>
-      <collision>
-      <origin xyz="0.0 0.0 0.0" rpy="1.5707 0 4.71" />
-      <geometry>
-        <mesh filename="package://two_wheel_mr/meshes/rplidar.dae" scale="0.001 0.001 0.001" />
-      </geometry>
-      </collision>
-    </link>
-    <joint name="${prefix}lidar_joint" type="fixed">
-      <parent link="${prefix}base_link" />
-      <child link="${prefix}lidar_link" />
-      <origin xyz="0.0 0 0.255" rpy="0 0 0" />
+    <link
+      name="${prefix}lidar_link">
+      <inertial>
+        <origin
+          xyz="-0.023581450658916 8.05046002083643E-09 0.00223779817490377"
+          rpy="0 0 0" />
+        <mass
+          value="0.189335150961536" />
+        <inertia
+          ixx="9.4126569435462E-05"
+          ixy="4.82701982803445E-11"
+          ixz="-2.33945223821742E-06"
+          iyy="0.000100748999349168"
+          iyz="1.86083776093011E-13"
+          izz="0.000140289739768048" />
+      </inertial>
+      <visual>
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