Commit message: add arm to URDF description

File: urdf/robot_description.urdf.xacro (robot description, xacro)
@@ -631,4 +631,476 @@
         xyz="0 1 0" />
     </joint>
+    <joint
+      name="${prefix}arm_base_joint"
+      type="fixed">
+      <origin
+        xyz="0 0 0.175"
+        rpy="0 0 0" />
+      <parent
+        link="${prefix}base_link" />
+      <child
+        link="${prefix}arm_base_link" />
+      <axis
+        xyz="0 -1 0" />
+      <limit
+        lower="0"
+        upper="0"
+        effort="0"
+        velocity="0" />
+    </joint>
+    <link
+      name="${prefix}arm_base_link">
+      <inertial>
+        <origin
+          xyz="-0.00031896 -0.00029673 0.042463"
+          rpy="0 0 0" />
+        <mass
+          value="1.6185" />
+        <inertia
+          ixx="0.0030836"
+          ixy="1.5354E-05"
+          ixz="-1.9315E-05"
+          iyy="0.0030825"
+          iyz="-1.7918E-05"
+          izz="0.0045209" />
+      </inertial>
+      <visual>
+        <origin
+          xyz="0 0 0"
+          rpy="0 0 0" />
+        <geometry>
+          <mesh
+            filename="package://fairino_description/meshes/fairino5_v6/base_link.STL" />
+        </geometry>
+        <material
+          name="${prefix}">
+          <color
+            rgba="0.89804 0.91765 0.92941 1" />
+        </material>
+      </visual>
+      <collision>
+        <origin
+          xyz="0 0 0"
+          rpy="0 0 0" />
+        <geometry>
+          <mesh
+            filename="package://fairino_description/meshes/fairino5_v6/base_link.STL" />
+        </geometry>
+      </collision>
+    </link>
+    <link
+      name="${prefix}shoulder_link">
+      <inertial>
+        <origin
+          xyz="5.0029E-07 -0.0040922 0.14629"
+          rpy="0 0 0" />
+        <mass
+          value="4.3771" />
+        <inertia
+          ixx="0.010731"
+          ixy="-8.0587E-09"
+          ixz="-3.6773E-08"
+          iyy="0.010408"
+          iyz="0.00012853"
+          izz="0.0081793" />
+      </inertial>
+      <visual>
+        <origin
+          xyz="0 0 0"
+          rpy="0 0 0" />
+        <geometry>
+          <mesh
+            filename="package://fairino_description/meshes/fairino5_v6/shoulder_link.STL" />
+        </geometry>
+        <material
+          name="${prefix}">
+          <color
+            rgba="0.89804 0.91765 0.92941 1" />
+        </material>
+      </visual>
+      <collision>
+        <origin
+          xyz="0 0 0"
+          rpy="0 0 0" />
+        <geometry>
+          <mesh
+            filename="package://fairino_description/meshes/fairino5_v6/shoulder_link.STL" />
+        </geometry>
+      </collision>
+    </link>
+    <joint
+      name="${prefix}j1"
+      type="revolute">
+      <origin
+        xyz="0 0 0"
+        rpy="0 0 0" />
+      <parent
+        link="${prefix}arm_base_link" />
+      <child
+        link="${prefix}shoulder_link" />
+      <axis
+        xyz="0 0 1" />
+      <limit
+        lower="-3.0543"
+        upper="3.0543"
+        effort="150"
+        velocity="3.15" />
+      <calibration
+        rising="0"
+        falling="0" />
+      <dynamics
+        damping="0"
+        friction="0" />
+      <safety_controller
+        soft_lower_limit="-3.0543"
+        soft_upper_limit="3.0543"
+        k_position="15"
+        k_velocity="10" />
+    </joint>
+    <link
+      name="${prefix}upperarm_link">
+      <inertial>
+        <origin
+          xyz="-0.2125 -5.7643E-09 0.1346"
+          rpy="0 0 0" />
+        <mass
+          value="14.458" />
+        <inertia
+          ixx="0.028392"
+          ixy="-1.337E-07"
+          ixz="-3.9895E-09"
+          iyy="0.4559"
+          iyz="4.214E-08"
+          izz="0.44974" />
+      </inertial>
+      <visual>
+        <origin
+          xyz="0 0 0"
+          rpy="0 0 0" />
+        <geometry>
+          <mesh
+            filename="package://fairino_description/meshes/fairino5_v6/upperarm_link.STL" />
+        </geometry>
+        <material
+          name="${prefix}">
+          <color
+            rgba="0.89804 0.91765 0.92941 1" />
+        </material>
+      </visual>
+      <collision>
+        <origin
+          xyz="0 0 0"
+          rpy="0 0 0" />
+        <geometry>
+          <mesh
+            filename="package://fairino_description/meshes/fairino5_v6/upperarm_link.STL" />
+        </geometry>
+      </collision>
+    </link>
+    <joint
+      name="${prefix}j2"
+      type="revolute">
+      <origin
+        xyz="0 0 0.152"
+        rpy="1.5708 0 0" />
+      <parent
+        link="${prefix}shoulder_link" />
+      <child
+        link="${prefix}upperarm_link" />
+      <axis
+        xyz="0 0 1" />
+      <limit
+        lower="-4.6251"
+        upper="1.4835"
+        effort="150"
+        velocity="3.15" />
+      <calibration
+        rising="0"
+        falling="0" />
+      <dynamics
+        damping="0"
+        friction="0" />
+      <safety_controller
+        soft_lower_limit="-4.6251"
+        soft_upper_limit="1.4835"
+        k_position="15"
+        k_velocity="10" />
+    </joint>
+    <link
+      name="${prefix}forearm_link">
+      <inertial>
+        <origin
+          xyz="-0.18793 -8.4503E-07 0.0066357"
+          rpy="0 0 0" />
+        <mass
+          value="7.6737" />
+        <inertia
+          ixx="0.0085096"
+          ixy="2.1613E-06"
+          ixz="-0.0068678"
+          iyy="0.16971"
+          iyz="3.7086E-08"
+          izz="0.16854" />
+      </inertial>
+      <visual>
+        <origin
+          xyz="0 0 0"
+          rpy="0 0 0" />
+        <geometry>
+          <mesh
+            filename="package://fairino_description/meshes/fairino5_v6/forearm_link.STL" />
+        </geometry>
+        <material
+          name="${prefix}">
+          <color
+            rgba="0.89804 0.91765 0.92941 1" />
+        </material>
+      </visual>
+      <collision>
+        <origin
+          xyz="0 0 0"
+          rpy="0 0 0" />
+        <geometry>
+          <mesh
+            filename="package://fairino_description/meshes/fairino5_v6/forearm_link.STL" />
+        </geometry>
+      </collision>
+    </link>
+    <joint
+      name="${prefix}j3"
+      type="revolute">
+      <origin
+        xyz="-0.425 0 0"
+        rpy="0 0 0" />
+      <parent
+        link="${prefix}upperarm_link" />
+      <child
+        link="${prefix}forearm_link" />
+      <axis
+        xyz="0 0 1" />
+      <limit
+        lower="-2.8274"
+        upper="2.8274"
+        effort="150"
+        velocity="3.15" />
+      <calibration
+        rising="0"
+        falling="0" />
+      <dynamics
+        damping="0"
+        friction="0" />
+      <safety_controller
+        soft_lower_limit="-2.8274"
+        soft_upper_limit="2.8274"
+        k_position="15"
+        k_velocity="10" />
+    </joint>
+    <link
+      name="${prefix}wrist1_link">
+      <inertial>
+        <origin
+          xyz="4.98E-07 -0.003754 0.097155"
+          rpy="0 0 0" />
+        <mass
+          value="1.6266" />
+        <inertia
+          ixx="0.00216"
+          ixy="4.888E-09"
+          ixz="3.1528E-08"
+          iyy="0.0015455"
+          iyz="3.7678E-05"
+          izz="0.0019902" />
+      </inertial>
+      <visual>
+        <origin
+          xyz="0 0 0"
+          rpy="0 0 0" />
+        <geometry>
+          <mesh
+            filename="package://fairino_description/meshes/fairino5_v6/wrist1_link.STL" />
+        </geometry>
+        <material
+          name="${prefix}">
+          <color
+            rgba="0.89804 0.91765 0.92941 1" />
+        </material>
+      </visual>
+      <collision>
+        <origin
+          xyz="0 0 0"
+          rpy="0 0 0" />
+        <geometry>
+          <mesh
+            filename="package://fairino_description/meshes/fairino5_v6/wrist1_link.STL" />
+        </geometry>
+      </collision>
+    </link>
+    <joint
+      name="${prefix}j4"
+      type="revolute">
+      <origin
+        xyz="-0.39501 0 0"
+        rpy="0 0 0" />
+      <parent
+        link="${prefix}forearm_link" />
+      <child
+        link="${prefix}wrist1_link" />
+      <axis
+        xyz="0 0 1" />
+      <limit
+        lower="-4.6251"
+        upper="1.4835"
+        effort="28"
+        velocity="3.2" />
+      <calibration
+        rising="0"
+        falling="0" />
+      <dynamics
+        damping="0"
+        friction="0" />
+      <safety_controller
+        soft_lower_limit="-4.6251"
+        soft_upper_limit="1.4835"
+        k_position="15"
+        k_velocity="10" />
+    </joint>
+    <link
+      name="${prefix}wrist2_link">
+      <inertial>
+        <origin
+          xyz="-4.5588E-07 0.0038617 0.098257"
+          rpy="0 0 0" />
+        <mass
+          value="1.5812" />
+        <inertia
+          ixx="0.0020612"
+          ixy="8.7064E-09"
+          ixz="-3.4742E-08"
+          iyy="0.0014477"
+          iyz="-2.8534E-05"
+          izz="0.0019573" />
+      </inertial>
+      <visual>
+        <origin
+          xyz="0 0 0"
+          rpy="0 0 0" />
+        <geometry>
+          <mesh
+            filename="package://fairino_description/meshes/fairino5_v6/wrist2_link.STL" />
+        </geometry>
+        <material
+          name="${prefix}">
+          <color
+            rgba="0.89804 0.91765 0.92941 1" />
+        </material>
+      </visual>
+      <collision>
+        <origins
+          xyz="0 0 0"
+          rpy="0 0 0" />
+        <geometry>
+          <mesh
+            filename="package://fairino_description/meshes/fairino5_v6/wrist2_link.STL" />
+        </geometry>
+      </collision>
+    </link>
+    <joint
+      name="${prefix}j5"
+      type="revolute">
+      <origin
+        xyz="0 0 0.1021"
+        rpy="1.5708 0 0" />
+      <parent
+        link="${prefix}wrist1_link" />
+      <child
+        link="${prefix}wrist2_link" />
+      <axis
+        xyz="0 0 1" />
+      <limit
+        lower="-3.0543"
+        upper="3.0543"
+        effort="28"
+        velocity="3.2" />
+      <calibration
+        rising="0"
+        falling="0" />
+      <dynamics
+        damping="0"
+        friction="0" />
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