Commit message: integrate moveit arm control
mostly copied from fairino5_v6_moveit2_config

File: urdf/drivetrain.urdf.xacro (robot description, xacro)
@@ -3,7 +3,10 @@
     <xacro:arg name="prefix" default="" />
     <xacro:arg name="use_mock_hardware" default="false" />
+    <xacro:arg name="initial_positions_file" default="$(find two_wheel_mr)/config/arm_init_positions.yaml" />
     <xacro:include filename="$(find two_wheel_mr)/urdf/robot_description.urdf.xacro" />
     <!-- Import ros2_control description -->
     <xacro:include filename="$(find kinco_diff_controller)/urdf/robot_control.urdf.xacro" />
+    <xacro:include filename="$(find two_wheel_mr)/urdf/fairino5_v6_robot.ros2_control.xacro" />
+    <!-- modified to allow choosing between using mock and actual hardware -->
     <xacro:robot prefix="$(arg prefix)" />
     <xacro:robot_control
@@ -11,3 +14,6 @@
         port="/dev/ttyS0" left_id="1" right_id="2"
         use_mock_hardware="$(arg use_mock_hardware)"/>
+    <xacro:fairino5_v6_robot_ros2_control
+        name="fairino5" initial_positions_file="$(arg initial_positions_file)"
+        use_mock_hardware="$(arg use_mock_hardware)"/>
 </robot>

File: urdf/robot_description.urdf.xacro (robot description, xacro)
@@ -42,10 +42,10 @@
       </collision>
     </link>
-    <link name="${prefix}base_footprint" />
+    <!-- <link name="${prefix}base_footprint" />
     <joint name="${prefix}base_joint" type="fixed">
-      <parent link="${prefix}${prefix}base_footprint" />
-      <child link="${prefix}${prefix}base_link" />
+      <parent link="${prefix}base_footprint" />
+      <child link="${prefix}base_link" />
       <origin xyz="0 0 0" rpy="0 0 0" />
-    </joint>
+    </joint> -->
     <link
       name="${prefix}base_scan">

Commit message: specify Fairino IP address as per latest frcobot_ros2 commit
only works if the github.com/itsmevjnk fork is used

File: urdf/drivetrain.urdf.xacro (robot description, xacro)
@@ -16,4 +16,5 @@
     <xacro:fairino5_v6_robot_ros2_control
         name="fairino5" initial_positions_file="$(arg initial_positions_file)"
+        address="192.168.58.2"
         use_mock_hardware="$(arg use_mock_hardware)"/>
 </robot>

File: urdf/fairino5_v6_robot.ros2_control.xacro (robot description, xacro)
@@ -1,5 +1,5 @@
 <?xml version="1.0"?>
 <robot xmlns:xacro="http://www.ros.org/wiki/xacro">
-    <xacro:macro name="fairino5_v6_robot_ros2_control" params="name initial_positions_file use_mock_hardware">
+    <xacro:macro name="fairino5_v6_robot_ros2_control" params="name initial_positions_file use_mock_hardware address">
         <xacro:property name="initial_positions" value="${xacro.load_yaml(initial_positions_file)['initial_positions']}"/>
         <ros2_control name="${name}" type="system">
@@ -7,4 +7,5 @@
                 <hardware>
                     <plugin>fairino_hardware/FairinoHardwareInterface</plugin>
+                    <param name="controller_ip">${address}</param>
                 </hardware>
             </xacro:unless>
